File: PCB/yui.kicad_pcb (KiCad board)
At the start: 4 copper layers, 45 x 75 mm, 77 parts, among them J1 Conn_Coaxial, J2 Conn_ARM_JTAG_SWD_10, J3 67068-8000, J4 PLR135/T9, J5 Conn_02x08_Odd_Even, J6 Conn_01x03, U1 STM32F765NIHx, U2 MIC5355-S4YMME, U3 NBA3N012C, U4 KC3225K24.0000C1GE00, U5 USB3300-EZK, U6 ICE40HX8K-BG121, U7 KC3225K22.5792C10E00, U8 KC3225K24.5760C10E00

Commit message: WIP changes
Other:
- net class Default removed
